Commit message: implementation: new cpp control scripts, prototyping cmd_vel publishing, hydrodynamics prototyping

File: src/auv_description/urdf/cube/plugins.xacro (robot description, xacro)
@@ -21,4 +21,22 @@
         <force_scale>1.0</force_scale>
         <torque_scale>1.0</torque_scale>
+        <force_topic>/auve1/force_body</force_topic>
+        <torque_topic>/auve1/torque_body</torque_topic>
+      </plugin>
+    </gazebo>
+  </xacro:macro>
+  <xacro:macro name="hydrodynamics_plugin" params="fluid_density">
+    <gazebo>
+      <plugin name="simple_hydrodynamics" filename="libsimple_hydrodynamics.so">
+        <link_name>${link_name}</link_name>
+        <!-- Water properties -->
+        <water_density>${fluid_density}</water_density>
+        <default_current>0 0 0</default_current>  <!-- world-frame m/s -->
+        <!-- Translational drag (body frame) -->
+        <linear_drag>20 20 20</linear_drag>               <!-- or try 20 20 20 -->
+        <quadratic_drag>550 550 550</quadratic_drag>   <!-- N/(m/s)^2 -->
+        <!-- Rotational drag (body frame) -->
+        <angular_drag>0 0 0</angular_drag>             <!-- or try 5 5 5 -->
+        <quadratic_angular_drag>137 137 137</quadratic_angular_drag> <!-- N·m/(rad/s)^2 -->
       </plugin>
     </gazebo>

Commit message: implementation: added prototype torpedo plugin

File: src/auv_description/urdf/cube/plugins.xacro (robot description, xacro)
@@ -26,5 +26,5 @@
     </gazebo>
   </xacro:macro>
-  <xacro:macro name="hydrodynamics_plugin" params="fluid_density">
+  <xacro:macro name="hydrodynamics_plugin" params="link_name fluid_density">
     <gazebo>
       <plugin name="simple_hydrodynamics" filename="libsimple_hydrodynamics.so">
@@ -42,3 +42,14 @@
     </gazebo>
   </xacro:macro>
+  <xacro:macro name="torpedo_plugin" params="link_name">
+    <gazebo>
+    <plugin name="auv_sim::TorpedoShooterPlugin" filename="libtorpedo_shooter.so">
+    <torpedo_sdf_path>$(find auv_description)/urdf/torpedo/torpedo1.sdf</torpedo_sdf_path>
+    <launcher_link>${link_name}</launcher_link>
+    <shoot_force>20</shoot_force>
+    <shoot_duration>0.1</shoot_duration>
+    <initial_velocity>3.0</initial_velocity>
+    </plugin>
+    </gazebo>
+  </xacro:macro>
 </robot>
