Commit message: implementation: fixed guppy urdf, implemented slider teleop

File: src/auv_description/urdf/guppy/guppytest1.urdf (robot description, URDF)
Before this commit: robot guppytest1, 9 links, 8 joints
Links:
- link thruster3M_link: mass 0 -> 0.17277
Joints:
- joint thruster0C_joint: axis 0 0 0 -> (none); origin xyz=-0.24536 0.27819 -0.019075 rpy=1.5708 0 -2.3562 -> xyz=0.27819 0.24536 -0.019075 rpy=1.5708 0 -3.9270
- joint thruster0M_joint: axis 0 0 0 -> (none); origin xyz=2.5E-05 0.2903 -0.013798 rpy=1.5708 1.5708 0 -> xyz=0.2903 -2.5E-05 -0.013798 rpy=1.5708 1.5708 -1.5708
- joint thruster1C_joint: axis 0 0 0 -> (none); origin xyz=0.24536 0.27819 -0.019025 rpy=-1.5708 0 -0.7854 -> xyz=0.27819 -0.24536 -0.019025 rpy=-1.5708 0 -2.3562
- joint thruster1M_joint: axis 0 0 0 -> (none); origin xyz=0.2649 -2.5E-05 -0.013798 rpy=0 1.5708 0 -> xyz=-2.5E-05 -0.2649 -0.013798 rpy=0 1.5708 -1.5708
- joint thruster2C_joint: axis 0 0 0 -> (none); origin xyz=0.24536 -0.27819 -0.019075 rpy=1.5708 0 0.7854 -> xyz=-0.27819 -0.24536 -0.019075 rpy=1.5708 0 -0.7854
- joint thruster2M_joint: axis 0 0 0 -> (none); origin xyz=-2.5E-05 -0.2903 -0.013798 rpy=1.5708 1.5708 0 -> xyz=-0.2903 2.5E-05 -0.013798 rpy=1.5708 1.5708 -1.5708
- joint thruster3C_joint: axis 0 0 0 -> (none); origin xyz=-0.24536 -0.27819 -0.019075 rpy=-1.5708 0 2.3562 -> xyz=-0.27819 0.24536 -0.019075 rpy=-1.5708 0 0.7854
- joint thruster3M_joint: axis 0 0 0 -> (none); origin xyz=-0.2649 2.5E-05 -0.013798 rpy=3.1416 1.5708 0 -> xyz=2.5E-05 0.2649 -0.013798 rpy=3.1416 1.5708 -1.5708

File: src/auv_description/urdf/guppy/plugins.xacro (robot description, xacro)
@@ -11,5 +11,5 @@
     </gazebo>
   </xacro:macro>
-  <!-- <xacro:macro name="wasd_plugin" params="link_name topic">
+  <xacro:macro name="wasd_plugin" params="link_name topic">
     <gazebo>
       <plugin name="wasd_body_thrust_plugin" filename="libwasd_body_thrust_plugin.so">
@@ -22,4 +22,4 @@
       </plugin>
     </gazebo>
-  </xacro:macro> -->
+  </xacro:macro>
 </robot>

Commit message: implementation: added rgbd to guppy

File: src/auv_description/urdf/guppy/guppytest1.urdf (robot description, URDF)
Before this commit: robot guppytest1, 9 links, 8 joints
Links:
- added link camera_link, mass 0.1; collision box size=0.10 0.06 0.04; visual box size=0.10 0.06 0.04
- added link camera_optical_frame
Joints:
- added joint camera_joint: type fixed, parent base_link, child camera_link, origin xyz=0.00 0.20 0.10 rpy=0 0 1.57079632679
- added joint camera_optical_joint: type fixed, parent camera_link, child camera_optical_frame, origin xyz=0 0 0 rpy=-1.57079632679 0 1.57079632679

File: src/auv_description/urdf/guppyExperimental/guppytest1Experimental.urdf (robot description, URDF)
Before this commit: robot guppytest1, 10 links, 9 joints
Links:
- added link camera_link, mass 0.1; collision box size=0.10 0.06 0.04; visual box size=0.10 0.06 0.04
- added link camera_optical_frame
Joints:
- added joint camera_joint: type fixed, parent base_link, child camera_link, origin xyz=0.00 0.20 0.10 rpy=0 0 1.57079632679
- added joint camera_optical_joint: type fixed, parent camera_link, child camera_optical_frame, origin xyz=0 0 0 rpy=-1.57079632679 0 1.57079632679

Commit message: implementation: added corner cameras

File: src/auv_description/urdf/guppy/guppytest1.urdf (robot description, URDF)
Before this commit: robot guppytest1, 11 links, 10 joints
Links:
- added link cam_fl_link, mass 0.05; collision box size=0.06 0.03 0.03; visual box size=0.06 0.03 0.03
- added link cam_fl_optical_frame
- added link cam_fr_link, mass 0.05; collision box size=0.06 0.03 0.03; visual box size=0.06 0.03 0.03
- added link cam_fr_optical_frame
- added link cam_rl_link, mass 0.05; collision box size=0.06 0.03 0.03; visual box size=0.06 0.03 0.03
- added link cam_rl_optical_frame
- added link cam_rr_link, mass 0.05; collision box size=0.06 0.03 0.03; visual box size=0.06 0.03 0.03
- added link cam_rr_optical_frame
Joints:
- added joint cam_fl_joint: type fixed, parent base_link, child cam_fl_link, origin xyz=0.25 0.18 0.10 rpy=0 0 0.78539816339
- added joint cam_fl_optical_joint: type fixed, parent cam_fl_link, child cam_fl_optical_frame, origin xyz=0 0 0 rpy=-1.57079632679 0 -1.57079632679
- added joint cam_fr_joint: type fixed, parent base_link, child cam_fr_link, origin xyz=0.25 -0.18 0.10 rpy=0 0 -0.78539816339
- added joint cam_fr_optical_joint: type fixed, parent cam_fr_link, child cam_fr_optical_frame, origin xyz=0 0 0 rpy=-1.57079632679 0 -1.57079632679
- added joint cam_rl_joint: type fixed, parent base_link, child cam_rl_link, origin xyz=-0.25 0.18 0.10 rpy=0 0 2.35619449019
- added joint cam_rl_optical_joint: type fixed, parent cam_rl_link, child cam_rl_optical_frame, origin xyz=0 0 0 rpy=-1.57079632679 0 -1.57079632679
- added joint cam_rr_joint: type fixed, parent base_link, child cam_rr_link, origin xyz=-0.25 -0.18 0.10 rpy=0 0 -2.35619449019
- added joint cam_rr_optical_joint: type fixed, parent cam_rr_link, child cam_rr_optical_frame, origin xyz=0 0 0 rpy=-1.57079632679 0 -1.57079632679

File: src/auv_description/urdf/guppyExperimental/guppytest1Experimental.urdf (robot description, URDF)
Before this commit: robot guppytest1, 12 links, 11 joints
Links:
- added link cam_fl_link, mass 0.05; collision box size=0.06 0.03 0.03; visual box size=0.06 0.03 0.03
- added link cam_fl_optical_frame
- added link cam_fr_link, mass 0.05; collision box size=0.06 0.03 0.03; visual box size=0.06 0.03 0.03
- added link cam_fr_optical_frame
- added link cam_rl_link, mass 0.05; collision box size=0.06 0.03 0.03; visual box size=0.06 0.03 0.03
- added link cam_rl_optical_frame
- added link cam_rr_link, mass 0.05; collision box size=0.06 0.03 0.03; visual box size=0.06 0.03 0.03
- added link cam_rr_optical_frame
Joints:
- added joint cam_fl_joint: type fixed, parent base_link, child cam_fl_link, origin xyz=0.25 0.18 0.10 rpy=0 0 0.78539816339
- added joint cam_fl_optical_joint: type fixed, parent cam_fl_link, child cam_fl_optical_frame, origin xyz=0 0 0 rpy=-1.57079632679 0 -1.57079632679
- added joint cam_fr_joint: type fixed, parent base_link, child cam_fr_link, origin xyz=0.25 -0.18 0.10 rpy=0 0 -0.78539816339
- added joint cam_fr_optical_joint: type fixed, parent cam_fr_link, child cam_fr_optical_frame, origin xyz=0 0 0 rpy=-1.57079632679 0 -1.57079632679
- added joint cam_rl_joint: type fixed, parent base_link, child cam_rl_link, origin xyz=-0.25 0.18 0.10 rpy=0 0 2.35619449019
- added joint cam_rl_optical_joint: type fixed, parent cam_rl_link, child cam_rl_optical_frame, origin xyz=0 0 0 rpy=-1.57079632679 0 -1.57079632679
- added joint cam_rr_joint: type fixed, parent base_link, child cam_rr_link, origin xyz=-0.25 -0.18 0.10 rpy=0 0 -2.35619449019
- added joint cam_rr_optical_joint: type fixed, parent cam_rr_link, child cam_rr_optical_frame, origin xyz=0 0 0 rpy=-1.57079632679 0 -1.57079632679

Commit message: implementation: added dvl to guppy, updated readme

File: src/auv_description/urdf/guppy/guppytest1.urdf (robot description, URDF)
Before this commit: robot guppytest1, 19 links, 18 joints
Links:
- added link dvl_link, mass 0.05; collision box size=0.03 0.03 0.03; visual box size=0.03 0.03 0.03
Joints:
- added joint dvl_joint: type fixed, parent base_link, child dvl_link, origin xyz=0.0 0.0 -0.20 rpy=0 0 0

File: src/auv_description/urdf/guppyExperimental/guppytest1Experimental.urdf (robot description, URDF)
Before this commit: robot guppytest1, 20 links, 19 joints
Links:
- added link dvl_link, mass 0.05; collision box size=0.03 0.03 0.03; visual box size=0.03 0.03 0.03
Joints:
- added joint dvl_joint: type fixed, parent base_link, child dvl_link, origin xyz=0.0 0.0 -0.20 rpy=0 0 0

Commit message: fix altimeter and imu

File: src/auv_description/urdf/guppy/guppytest1.urdf (robot description, URDF)
Before this commit: robot guppytest1, 20 links, 19 joints
Links:
- added link imu_link, mass 0.01; collision box size=0.01 0.01 0.01; visual box size=0.01 0.01 0.01
Joints:
- added joint imu_joint: type fixed, parent base_link, child imu_link, origin xyz=0 0 0.05 rpy=0 0 0

Commit message: save changes

File: src/auv_description/urdf/guppy/guppytest1.urdf (robot description, URDF)
Before this commit: robot guppytest1, 21 links, 20 joints
Joints:
- joint thruster0M_joint: origin xyz=0.2903 -2.5E-05 -0.013798 rpy=1.5708 1.5708 -1.5708 -> xyz=0.2903 0 -0.013798 rpy=1.5708 1.5708 -1.5708
- joint thruster1M_joint: origin xyz=-2.5E-05 -0.2649 -0.013798 rpy=0 1.5708 -1.5708 -> xyz=0 -0.2649 -0.013798 rpy=0 1.5708 -1.5708
- joint thruster2M_joint: origin xyz=-0.2903 2.5E-05 -0.013798 rpy=1.5708 1.5708 -1.5708 -> xyz=-0.2903 0 -0.013798 rpy=1.5708 1.5708 -1.5708
- joint thruster3M_joint: origin xyz=2.5E-05 0.2649 -0.013798 rpy=3.1416 1.5708 -1.5708 -> xyz=0 0.2649 -0.013798 rpy=3.1416 1.5708 -1.5708

Commit message: updated stuff

File: src/auv_description/urdf/guppy/guppytest1.urdf (robot description, URDF)
Before this commit: robot guppytest1, 21 links, 20 joints
Links:
- link cam_fl_link: mass 0.05 -> 0
- link cam_fr_link: mass 0.05 -> 0
- link cam_rl_link: mass 0.05 -> 0
- link cam_rr_link: mass 0.05 -> 0
- link camera_link: mass 0.1 -> 0
- link dvl_link: mass 0.05 -> 0
Joints:
- joint dvl_joint: origin xyz=0.0 0.0 -0.20 rpy=0 0 0 -> xyz=0.0 0.0 -0.05 rpy=0 0 0

Commit message: fix: some changes

File: src/auv_description/urdf/guppy/guppytest1.urdf (robot description, URDF)
Before this commit: robot guppytest1, 21 links, 20 joints
Links:
- link base_link: mass 12.294 -> 20

Commit message: feat: working sim

File: src/auv_description/urdf/guppy/guppytest1.urdf (robot description, URDF)
Before this commit: robot guppytest1, 21 links, 20 joints
Links:
- link imu_link: mass 0.01 -> 0
- link thruster0C_link: mass 0.17277 -> 0
- link thruster0M_link: mass 0.17279 -> 0
- link thruster1C_link: mass 0.17277 -> 0
- link thruster1M_link: mass 0.17279 -> 0
- link thruster2C_link: mass 0.17277 -> 0
- link thruster2M_link: mass 0.17279 -> 0
- link thruster3C_link: mass 0.17277 -> 0
- link thruster3M_link: mass 0.17277 -> 0
